Commit message: added in the target but still needs debugging

File: arm_description/urdf/arm_gazebo.urdf.xacro (robot description, xacro)
@@ -88,4 +88,6 @@
     </sensor>
   </gazebo>
+  <gazebo reference="target">
+  </gazebo>
   <link name="dummy_link"/>
    <!--Dummy Link-->
@@ -340,3 +342,15 @@
     <origin xyz="0.0 0.0 0.0" rpy="0.0 0.0 0.0" />
   </joint>
+  <joint name="target_joint" type="fixed">
+    <parent link="world"/>
+    <child link="target"/>
+    <origin xyz="1.5 1.5 0" rpy="1.5 1.5 0" />
+  </joint>
+  <link name="target">
+    <visual>
+      <geometry>
+        <box size="1 1 0.001"/>
+      </geometry>
+    </visual>
+  </link>
 </robot>

Commit message: got the target to a nice location and orientation in gazebo

File: arm_description/urdf/arm_gazebo.urdf.xacro (robot description, xacro)
@@ -90,4 +90,10 @@
   <gazebo reference="target">
   </gazebo>
+  <material name="blue">
+    <color rgba="0 0 0.8 1"/>
+  </material>
+  <material name="white">
+    <color rgba="1 1 1 1"/>
+  </material>
   <link name="dummy_link"/>
    <!--Dummy Link-->
@@ -345,12 +351,18 @@
     <parent link="world"/>
     <child link="target"/>
-    <origin xyz="1.5 1.5 0" rpy="1.5 1.5 0" />
+    <origin xyz="1 0 0.25" rpy="0 1.571 0" />
   </joint>
   <link name="target">
     <visual>
       <geometry>
-        <box size="1 1 0.001"/>
-      </geometry>
-    </visual>
+        <box size="0.25 0.25 0.00001"/>
+      </geometry>
+      <material name="blue"/>
+    </visual>
+    <inertial>
+      <mass value="1" />
+      <origin xyz="0 0 0" rpy="0 0 0" />
+      <inertia ixx="1e-6" ixy="0" ixz="0" iyy="1e-6" iyz="0" izz="1e-6" />
+    </inertial>
   </link>
 </robot>

Commit message: got the target colour working in gazebo

File: arm_description/urdf/arm_gazebo.urdf.xacro (robot description, xacro)
@@ -89,4 +89,5 @@
   </gazebo>
   <gazebo reference="target">
+    <material>Gazebo/Blue</material>
   </gazebo>
   <material name="blue">

Commit message: removed the urdf target object as it is redundant

File: arm_description/urdf/arm_gazebo.urdf.xacro (robot description, xacro)
@@ -88,13 +88,4 @@
     </sensor>
   </gazebo>
-  <gazebo reference="target">
-    <material>Gazebo/Blue</material>
-  </gazebo>
-  <material name="blue">
-    <color rgba="0 0 0.8 1"/>
-  </material>
-  <material name="white">
-    <color rgba="1 1 1 1"/>
-  </material>
   <link name="dummy_link"/>
    <!--Dummy Link-->
@@ -349,21 +340,3 @@
     <origin xyz="0.0 0.0 0.0" rpy="0.0 0.0 0.0" />
   </joint>
-  <joint name="target_joint" type="fixed">
-    <parent link="world"/>
-    <child link="target"/>
-    <origin xyz="1 0 0.25" rpy="0 1.571 0" />
-  </joint>
-  <link name="target">
-    <visual>
-      <geometry>
-        <box size="0.25 0.25 0.00001"/>
-      </geometry>
-      <material name="blue"/>
-    </visual>
-    <inertial>
-      <mass value="1" />
-      <origin xyz="0 0 0" rpy="0 0 0" />
-      <inertia ixx="1e-6" ixy="0" ixz="0" iyy="1e-6" iyz="0" izz="1e-6" />
-    </inertial>
-  </link>
 </robot>
